File: pcb/Untitled.sch (KiCad schematic (older format))
At the start: 13 parts

Commit message: added pcb schematics
Parts:
- removed SW? (x6): MX-with-LED, symbol keebio:MX-with-LED
- added SW? (x6): MX-with-LED, symbol keebio:MX-with-LED
Connections:
- net at U?.25 (B7): now also SW?.1, SW?.1, SW?.1, SW?.1, SW?.1
- net at U?.26 (D5): now also SW?.1, SW?.1, SW?.1
- net at U?.27 (C7): now also SW?.2, SW?.4, SW?.4, SW?.4, U?.4 (GND), U?.7 (4/PD4), SW?.2, SW?.2, SW?.4, SW?.4, SW?.4, SW?.4, SW?.4, SW?.4
- net at U?.5 (2/PD1): now also SW?.2, SW?.2, SW?.2
- net at U?.6 (3/PD0): now also SW?.2, SW?.2, SW?.2
- net at U?.8 (5/PC6): now also SW?.2, SW?.2
- net at U?.9 (6/PD7): now also SW?.2
- net at SW?.1: now also SW?.1, SW?.1, SW?.1
- net +5V: no longer names the net of U?.21 (VCC)
Other:
- moved on the sheet: SW?, U?

Commit message: updated firmware and pcb schematics
Parts:
- removed SW? (x12): MX-with-LED, symbol keebio:MX-with-LED
- removed U?: Elite-C, symbol keebio:Elite-C
- added D? (x12): D_Small, symbol Device:D_Small
- added MX? (x12): MX-LED, symbol MX_Alps_Hybrid:MX-LED
- added U?: Elite-C, symbol keebio:Elite-C
Connections:
- net labels added: col1, col2, col3, row1, row2, row3, row4, row5
- wire segments 88 -> 41

Commit message: Created PCB with Elite-C usage in mind. The hardware now supports led.
Parts:
- D1, D10, D11, D12, D2, D3, D4, D5, D6, D7, D8, D9: renamed from D?; footprint (none) -> Diode_SMD:D_0805_2012Metric
- MX1, MX2: renamed from MX?; footprint (none) -> MX_Only:MXOnly-1.5U
- MX10, MX11, MX12, MX3, MX4, MX5, MX6, MX7, MX8, MX9: renamed from MX?; footprint (none) -> MX_Only:MXOnly-1U
- U1: renamed from U?; footprint (none) -> Keebio-Parts:Elite-C
Connections:
- net labels added: gnd, led1, led2, led3, led4, led5, led6, led7, led8, led9
- wire segments 41 -> 77
