File: pcb/rev1/IKIDS.kicad_pcb (KiCad board)
At the start: 2 copper layers, 142.9 x 95.3 mm, 25 parts, among them U1 Elite-C

Commit message: Added logo to PCB
Other:
- board text added: "Huskeyboards-IKIDS Rev 1.0"
